File: content/electrical/Baby slip ring/Ring Side/Ring Side.kicad_pcb (KiCad board)
At the start: 2 copper layers, 57.5 x 57.5 mm, 8 parts, among them J1 USB4105-GF-A, U1 2_Wire_Ring

Commit message: first save of babyslipring
Parts:
- R1, R2, R3: value 56.2k -> 5.1k
- moved R3 4.64 mm to (172.7, 99.1), turned to 180 degrees
- moved R2 3.90 mm to (167.6, 99.1)
- moved R4 1.35 mm to (172.7, 83.8)
- moved R1 0.68 mm to (167.6, 83.8)
Connections:
- R1 pad 1: Net-(J1-PadS1) -> GND
- R1 pad 2: GND -> Net-(J1-PadS1)
- R2 pad 2: VCC -> GND
- R3 pad 2: VCC -> GND
Routing:
- net VCC: track 23.6 -> 15.0 mm, vias 2 -> 4
- net Net-(J1-PadA5): track 13.3 -> 7.75 mm
- net Net-(R4-Pad1): track 18.7 -> 23.0 mm
- net GND: track 10.4 -> 13.6 mm, vias 2 -> 3
- net Net-(J1-PadB5): track 9.84 -> 11.6 mm
